File: v1.0/thingBot-LoRa_v1P0.kicad_pcb (KiCad board)
At the start: 2 copper layers, 24.4 x 32.9 mm, 45 parts, among them U1 EDGE_SMA, U2 RFM92/95, U3 XBEE_MODULE

Commit message: Final layout done and Gerbers generated
Other:
- board text added: "DIO0"
- board text added: "DIO1"
- board text added: "DIO2"
- board text added: "DIO3"
- board text added: "DIO4"
- board text added: "DIO5"
- board text added: "GND"
- board text added: "SCK"
- board text added: "SIMO"
- board text added: "SOMI"
- board text added: "VIN"
- board text added: "nCS"
- board text added: "nRST"
Changed lines of the file:
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@@
     (area 170.939999 97.939999 195.420001 130.970001)
     (thickness 1.6)
-    (drawings 12)
+    (drawings 26)
     (tracks 110)
     (zones 0)
@@
     (tags "capacitor 0805")
     (attr smd)
-    (fp_text reference C2 (at 0.05 1.52 180) (layer F.SilkS)
-      (effects (font (size 1 1) (thickness 0.15)))
-    )
-    (fp_text value 0.1uF (at 0 2.1 180) (layer F.Fab)
-      (effects (font (size 1 1) (thickness 0.15)))
+    (fp_text reference C2 (at 0 2.14 180) (layer F.SilkS)
+      (effects (font (size 1 1) (thickness 0.15)))
+    )
+    (fp_text value 0.1uF (at 0.04 1.27 180) (layer F.Fab)
+      (effects (font (size 0.5 0.5) (thickness 0.09)))
     )
     (fp_line (start -1 0.625) (end -1 -0.625) (layer F.Fab) (width 0.15))
@@
       (effects (font (size 1 1) (thickness 0.15)))
     )
-    (fp_text value 1K (at 4.16 0.02 270) (layer F.Fab)
-      (effects (font (size 1 1) (thickness 0.15)))
+    (fp_text value 1K (at -2.68 -0.02 270) (layer F.Fab)
+      (effects (font (size 0.5 0.5) (thickness 0.09)))
     )
     (fp_line (start -1 0.625) (end -1 -0.625) (layer F.Fab) (width 0.1))
@@
   (module Xbee:Xbee_mod locked (layer F.Cu)
     (at 172.18 105.23)
-    (fp_text reference U3 (at 11 2) (layer F.SilkS)
-      (effects (font (size 1 1) (thickness 0.15)))
-    )
-    (fp_text value XBEE_MODULE (at 11 0) (layer F.Fab)
-      (effects (font (size 1 1) (thickness 0.15)))
+    (fp_text reference U3 (at 11 2) (layer B.SilkS)
+      (effects (font (size 1 1) (thickness 0.15)) (justify mirror))
+    )
+    (fp_text value XBEE_MODULE (at 10.82 0.17) (layer B.SilkS)
+      (effects (font (size 1 1) (thickness 0.15)) (justify mirror))
     )
     (fp_line (start -1.19 -0.7) (end -1.19 25.71) (layer F.SilkS) (width 0.15))
@@
       (effects (font (size 1 1) (thickness 0.15)))
     )
-    (fp_text value POWER (at -5 -1.4 90) (layer F.Fab)
-      (effects (font (size 1 1) (thickness 0.15)))
+    (fp_text value POWER (at -0.01 2.52 90) (layer F.Fab)
+      (effects (font (size 0.5 0.5) (thickness 0.09)))
     )
     (fp_line (start -0.4 -0.3) (end -0.4 0.3) (layer F.Fab) (width 0.15))
@@
   (module Temp:RFM92_95_96_98 (layer B.Cu)
     (at 175.3 121.2)
-    (fp_text reference U2 (at 8 -6) (layer B.SilkS)
+    (fp_text reference U2 (at 7.23 -6.19) (layer B.SilkS)
       (effects (font (size 1 1) (thickness 0.15)) (justify mirror))
     )
@@
     (tags "capacitor 0805")
     (attr smd)
-    (fp_text reference C1 (at -0.01 1.5 180) (layer F.SilkS)
-      (effects (font (size 1 1) (thickness 0.15)))
-    )
-    (fp_text value 15nF (at 4.58 2.69 180) (layer F.Fab)
-      (effects (font (size 1 1) (thickness 0.15)))
+    (fp_text reference C1 (at -1.4 1.18 180) (layer F.SilkS)
+      (effects (font (size 0.7 0.7) (thickness 0.1)))
+    )
+    (fp_text value 15nF (at 0.13 1.24 180) (layer F.Fab)
+      (effects (font (size 0.5 0.5) (thickness 0.09)))
     )
     (fp_line (start -1 0.625) (end -1 -0.625) (layer F.Fab) (width 0.15))
@@
       (effects (font (size 1 1) (thickness 0.15)))
     )
-    (fp_text value 1K (at 0 2.1 180) (layer F.Fab)
-      (effects (font (size 1 1) (thickness 0.15)))
+    (fp_text value 1K (at -1.5 -1.49 180) (layer F.Fab)
+      (effects (font (size 0.5 0.5) (thickness 0.09)))
     )
     (fp_line (start -1 0.625) (end -1 -0.625) (layer F.Fab) (width 0.1))
@@
       (effects (font (size 0.5 0.5) (thickness 0.11)))
     )
-    (fp_text value RESET (at -5.3 2.89) (layer F.Fab)
-      (effects (font (size 1 1) (thickness 0.15)))
+    (fp_text value RESET (at 2.54 0.28 90) (layer F.Fab)
+      (effects (font (size 0.5 0.5) (thickness 0.09)))
     )
     (fp_line (start -2.4 1.65) (end 2.4 1.65) (layer F.CrtYd) (width 0.05))
@@
       (effects (font (size 1 1) (thickness 0.15)))
     )
-    (fp_text value EDGE_SMA (at -7.3 3.1 360) (layer F.Fab)
+    (fp_text value EDGE_SMA (at -6.76 2.62 360) (layer F.Fab)
       (effects (font (size 1 1) (thickness 0.15)))
     )
@@
       (effects (font (size 1 1) (thickness 0.15)))
     )
-    (fp_text value WIRE_ANT (at -0.635 3.81) (layer F.Fab)
+    (fp_text value WIRE_ANT (at 4.8 0.22) (layer F.Fab)
       (effects (font (size 1 1) (thickness 0.15)))
     )
@@
     )
   )
+  (gr_circle (center 174.34 122.32) (end 174.6 122.48) (layer B.SilkS) (width 0.2))
+  (gr_text DIO4 (at 191.85 123.23) (layer F.SilkS)
+    (effects (font (size 0.7 0.7) (thickness 0.175)))
+  )
+  (gr_text DIO5 (at 192.04 115.23) (layer F.SilkS)
+    (effects (font (size 0.7 0.7) (thickness 0.175)))
+  )
+  (gr_text DIO3 (at 192.01 111.23) (layer F.SilkS)
+    (effects (font (size 0.7 0.7) (thickness 0.175)))
+  )
+  (gr_text DIO2 (at 192.02 109.23) (layer F.SilkS)
+    (effects (font (size 0.7 0.7) (thickness 0.175)))
+  )
+  (gr_text DIO1 (at 192.04 107.23) (layer F.SilkS)
+    (effects (font (size 0.7 0.7) (thickness 0.175)))
+  )
+  (gr_text DIO0 (at 192.04 105.23) (layer F.SilkS)
+    (effects (font (size 0.7 0.7) (thickness 0.175)))
+  )
+  (gr_text VIN (at 174.4 105.23) (layer F.SilkS)
+    (effects (font (size 0.7 0.7) (thickness 0.175)))
+  )
+  (gr_text GND (at 174.26 123.23) (layer F.SilkS)
+    (effects (font (size 0.7 0.7) (thickness 0.175)))
+  )
+  (gr_text SIMO (at 174.23 121.23) (layer F.SilkS)
+    (effects (font (size 0.7 0.7) (thickness 0.175)))
+  )
+  (gr_text "nCS\n" (at 174.21 117.23) (layer F.SilkS)
+    (effects (font (size 0.7 0.7) (thickness 0.175)))
+  )
+  (gr_text SCK (at 174.23 115.23) (layer F.SilkS)
+    (effects (font (size 0.7 0.7) (thickness 0.175)))
+  )
+  (gr_text nRST (at 174.23 113.23) (layer F.SilkS)
+    (effects (font (size 0.7 0.7) (thickness 0.175)))
+  )
+  (gr_text SOMI (at 174.29 111.23) (layer F.SilkS)
+    (effects (font (size 0.7 0.7) (thickness 0.175)))
+  )
   (gr_text "32.94 x 24.38 mm" (at 151.83 97.47) (layer Dwgs.User)
     (effects (font (size 0.7 0.7) (thickness 0.15)))
@@
     (effects (font (size 0.5 0.5) (thickness 0.1)))
   )
-  (gr_text "thingBot-LoRa\n         v1.0" (at 183.83 111.91) (layer F.SilkS)
-    (effects (font (size 1.5 1.5) (thickness 0.3)))
+  (gr_text "thingBot-LoRa\n         v1.0" (at 183.31 111.95) (layer F.SilkS)
+    (effects (font (size 1.2 1.2) (thickness 0.2)))
   )
   (gr_line (start 195.37 104.51) (end 195.37 130.92) (layer Edge.Cuts) (width 0.1))
